File: Hardware/SO4R_Interlock/SO4R_Interlock.kicad_sch (KiCad schematic)
At the start: 120 parts, among them J1 USB-C 2.0 16P, J2 USB-C 2.0 16P, J3 USB-C 2.0 16P, J4 USB-C 2.0 16P, J5 8P8C_LED_Shielded_x4, J7 Header 1x3, U1 FT230XS, U10 TPD4E02B04DQA, U11 TPD4E02B04DQA, U12 TPD4E02B04DQA, U2 FT230XS, U3 74LVC1G07, U4 AVR32DB48x-xPT, U5 FT230XS, U6 FT230XS, U7 74LVC1G07, U8 74LVC1G07, U9 TPD4E02B04DQA

Commit message: Ordered V1 of Transfer Relay boards and Interlock boards and assembly
Parts:
- added C18, C19, C21, C22: .1u, Capacitor_SMD:C_0402_1005Metric, symbol Device:C_Small
- added J6: RJ45_LED_Shielded, Connector_RJ:RJ45_Amphenol_RJHSE538X, symbol Connector:RJ45_LED_Shielded
- added Q1, Q2, Q3, Q4, Q5, Q6, Q7, Q8: 2N7002, Package_TO_SOT_SMD:SOT-23, symbol Transistor_FET:2N7002
- added R25, R26: 1K, Resistor_SMD:R_0402_1005Metric, symbol Device:R_Small_US
- C24: renamed from C35; value .01 -> .1u
- C25: renamed from C28; value .01 -> .1u
- C26: renamed from C20; value .01 -> .1u
- C27: renamed from C25; value .01 -> .1u
- C28: renamed from C29; value .01 -> .1u
- C29: renamed from C30; value .01 -> .1u
- C30: renamed from C22; value .01 -> .1u
- C31: renamed from C24; value .01 -> .1u
- C32, C33: value .01 -> .1u
- C34: renamed from C27; value .01 -> .1u
- C35: renamed from C23; value .01 -> .1u
- C36: renamed from C31; value .01 -> .1u
- C37: renamed from C34; value .01 -> .1u
- C38: renamed from C26; value .01 -> .1u
- C39: renamed from C19; value .01 -> .1u
- D5: renamed from D13; value D_Schottky -> RBQ161QS-40
- R41: renamed from R27; value 33 -> 1K
- renumbered C14 to C1, C12 to C10, C16 to C11, C8 to C12, C17 to C13, C15 to C14, C9 to C15, C10 to C16, C21 to C17, C6 to C2, C11 to C20, C13 to C23, C2 to C4, C18 to C5, C5 to C6, C4 to C7, C1 to C8, C7 to C9, D15 to D1, D11 to D10, D6 to D11, D4 to D12, D3 to D13, D2 to D14, D8 to D15, D12 to D2, D5 to D3, D9 to D4, D7 to D6, D1 to D7, D14 to D8, D10 to D9, FB3 to FB1, FB1 to FB3, J4 to J1, J3 to J2, J1 to J3, J2 to J4, J7 to J5, J5 to J7, R8 to R1, R22 to R10, R23 to R11, R20 to R12, R21 to R13, R11 to R14, R18 to R15, R13 to R16, R12 to R17, R14 to R18, R16 to R19, R7 to R2, R10 to R20, R15 to R21, R24 to R22, R19 to R23, R17 to R24, R47 to R27, R43 to R28, R42 to R29, R6 to R3, R41 to R30, R40 to R31, R39 to R32, R38 to R33, R37 to R34, R28 to R35, R29 to R36, R30 to R37, R31 to R38, R32 to R39, R5 to R4, R33 to R40, R25 to R42, R44 to R43, R48 to R44, R46 to R45, R45 to R46, R35 to R47, R34 to R48, R26 to R49, R4 to R5, R36 to R50, R3 to R6, R2 to R7, R1 to R8, U5 to U1, U11 to U10, U10 to U11, U9 to U12, U6 to U2, U1 to U3, U2 to U4, U8 to U5, U7 to U6, U3 to U7, U4 to U8, U12 to U9
Connections:
- net GND: now also J7.11, J7.21, J7.23, J7.33, J7.35, J7.45, J7.47, J7.9, C18.1, C19.1, C21.1, C22.1, J6.11, J6.2, J6.4, J6.6, J6.8, J6.9, J6.SH, Q1.2 (S), Q2.2 (S), Q3.2 (S), Q4.2 (S), Q5.2 (S), Q6.2 (S), Q7.2 (S), Q8.2 (S); no longer J7.10, J7.12, J7.22, J7.24, J7.34, J7.36, J7.46, J7.48
- net PTT1: now also U8.23 (PD3), Q5.1 (G); no longer R40.1, U12.2 (IO2), U8.22 (PD2)
- net PTT2: now also Q8.1 (G); no longer R36.1, U11.2 (IO2)
- net PTT3: now also Q7.1 (G); no longer R32.1, U10.2 (IO2)
- net PTT4: now also Q6.1 (G); no longer R28.1, U9.2 (IO2)
- net SPR1: now also U8.21 (PD1); no longer U8.20 (PD0)
- net TX1_LED: now also U8.20 (PD0); no longer U8.19 (PC7)
- net TX2_LED: now also R47.2; no longer R47.1
- net at R48.1: now also J7.24; no longer J7.23
- net at R45.1: now also J7.34; no longer J7.33
- net at R46.1: now also J7.36; no longer J7.35
- net TX0: now reaches U8.12 (PC2)
- net TX0: now also R25.2
- net RLY1: now reaches U8.13 (PC3)
- net RLY1: now also Q4.1 (G)
- net RLY2: now reaches U8.16 (PC4)
- net RLY2: now also Q3.1 (G)
- net RLY3: now reaches U8.17 (PC5)
- net RLY3: now also Q2.1 (G)
- net RLY4: now reaches U8.18 (PC6)
- net RLY4: now also Q1.1 (G)
- net at R43.1: now also J7.46; no longer J7.45
- net at R49.1: now also J7.10; no longer J7.9
- net at R50.1: now also J7.12; no longer J7.11
- net at R44.1: now also J7.48; no longer J7.47
- net KEY1 renamed KEY1\
- net KEY1\: now also U8.22 (PD2); no longer U8.21 (PD1)
- net KEY2 renamed KEY2\
- net KEY3 renamed KEY3\
- net KEY4 renamed KEY4\
- new net: J7.22, R47.1
- new net: C21.2, J6.3, Q3.3 (D)
- new net: C19.2, J6.5, Q2.3 (D)
- new net: C22.2, J6.1, Q4.3 (D)
- new net: C18.2, J6.7, Q1.3 (D)
- new net: J6.12, R26.1
- new net: J6.10, R25.1
- new net PTT1\: Q5.3 (D), R40.1, U12.2 (IO2)
- new net PTT2\: Q8.3 (D), R36.1, U11.2 (IO2)
- new net PTT3\: Q7.3 (D), R32.1, U10.2 (IO2)
- new net PTT4\: Q6.3 (D), R28.1, U9.2 (IO2)
- new net TX1: R26.2, U8.19 (PC7)
- no-connect marks 36 -> 30
Other:
- moved on the sheet: C1, C10, C11, C12, C13, C14, C15, C16, C17, C2, C20, C23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

Commit message: Added drilling dimensions for Transfer Relay enclosure Added ethernet cable color codes to schematic, validated that part Validated KEY/ input to interlock works Validated KEY/ input inhibits lower priority radio and lites Inhibit LED Added rippling LED's to setup() code
Other:
- note added: "BLU/WHT"
- note added: "BRN/WHT"
- note added: "GRN/WHT"
- note added: "ORG/WHT"
- note added: "SO4R Interlock - One SSB/CW radio with operator - Three radios for FT8 Radio Interface - PTT/, to radio, open drain pulldown 60V 1A - KEY/, from radio, input, pullup - SPR, undefined, output, low - CAT, optional, control radio from USB, growth option USB interface for port 1, FTDI FX230 - TXD, RXD used for programming and serial comms, no CAT - RTS/, CTS/, routed to MCU, not used for SSB/CW radio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"
- note removed: "SO4R Interlock - SSB/CW radio with operator - Up to 3 radios for FT8 Radio Interface - PTT, to radio - KEY, from radio - SPR, undefined, growth option - CAT, optional, control radio from USB, growth option USB Interface FTDI FX230 USB serial - TXD, RXD, optional, control radio, growth option - RTS, to MCU, signals PC wants to transmit - CTS, to MCU, undefined, growth option - TXDEN, output to con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"
- moved on the sheet: C26, C27, C30, C31, C34, C35, C38, C39, J7A, J7B, Q5, Q6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
